File: KiCAD/thermal.kicad_sch (KiCad schematic)
At the start: 20 parts, among them J14 10k NTC, J15 10k NTC, J16 EN_NTC_B, J17 EN_NTC_A, J18 FAN, J19 FAN, M1 24V, M3 24V, Q10 AO3400A, U13 VOS618A-3T

Commit message: Sync KiCAD project
Forgot to push this earlier
Parts:
- C37, C38: LCSC Part (none) -> C14663
- D2, D9: LCSC Part (none) -> C14996
- R33: LCSC Part (none) -> C25076
- R34, R36, R38: LCSC Part (none) -> C25744
- R35: LCSC Part (none) -> C23204
Changed lines of the file:
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@@
 	(text "EL357N(A)(TA)-G needs 330R input resistor"
 		(exclude_from_sim no)
-		(at 39.37 62.23 0)
+		(at 123.19 -21.59 0)
 		(effects
 			(font
@@
 			)
 		)
+		(property "LCSC Part" "C25744"
+			(at 109.22 77.47 0)
+			(effects
+				(font
+					(size 1.27 1.27)
+				)
+				(hide yes)
+			)
+		)
 		(pin "1"
 		)
@@
 			)
 		)
+		(property "LCSC Part" "C14663"
+			(at 96.52 160.02 0)
+			(effects
+				(font
+					(size 1.27 1.27)
+				)
+				(hide yes)
+			)
+		)
 		(pin "1"
 		)
@@
 			)
 		)
+		(property "LCSC Part" "C14996"
+			(at 148.59 48.26 90)
+			(effects
+				(font
+					(size 1.27 1.27)
+				)
+				(hide yes)
+			)
+		)
 		(pin "2"
 		)
@@
 			)
 		)
+		(property "LCSC Part" "C23204"
+			(at 69.85 60.96 0)
+			(effects
+				(font
+					(size 1.27 1.27)
+				)
+				(hide yes)
+			)
+		)
 		(pin "1"
 		)
@@
 			)
 		)
+		(property "LCSC Part" "C25744"
+			(at 102.87 148.59 0)
+			(effects
+				(font
+					(size 1.27 1.27)
+				)
+				(hide yes)
+			)
+		)
 		(pin "1"
 		)
@@
 			)
 		)
+		(property "LCSC Part" "C14663"
+			(at 96.52 127 0)
+			(effects
+				(font
+					(size 1.27 1.27)
+				)
+				(hide yes)
+			)
+		)
 		(pin "1"
 		)
@@
 			)
 		)
+		(property "LCSC Part" "C14996"
+			(at 148.59 69.85 90)
+			(effects
+				(font
+					(size 1.27 1.27)
+				)
+				(hide yes)
+			)
+		)
 		(pin "2"
 		)
@@
 			)
 		)
+		(property "LCSC Part" "C25076"
+			(at 101.6 71.12 90)
+			(effects
+				(font
+					(size 1.27 1.27)
+				)
+				(hide yes)
+			)
+		)
 		(pin "1"
 		)
@@
 			(at 102.87 115.57 0)
 			(effects
+				(font
+					(size 1.27 1.27)
+				)
+				(hide yes)
+			)
+		)
+		(property "LCSC Part" "C25744"
+			(at 102.87 115.57 0)
+			(effects

Commit message: Add M3 mounting holes, Fix DRC Errors, Merge L3 Quiet Power GND Fills
Parts:
- added H1, H2, H3, H4, H5, H6, H7, H8: MountingHole, MountingHole:MountingHole_3.2mm_M3, symbol Mechanical:MountingHole

Commit message: Fixed silly miswired CAN transceivers
Other:
- note added: "M3 MOUNTING HOLES"
Changed lines of the file:
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@@
+		)
+	)
+	(text "M3 MOUNTING HOLES"
+		(exclude_from_sim no)
+		(at 241.3 66.04 0)
+		(effects
+			(font
+				(size 1.27 1.27)
+			)
 		)
 	)
